Commit message: Synchronization

File: src/slambot_description/urdf/slambot_gz_urdf.xacro (robot description, xacro)
@@ -4,5 +4,4 @@
                   value="$(find slambot_description)"/>
   <xacro:include filename="${slambot_description_share}/urdf/materials.xacro"/>
-  <xacro:include filename="${slambot_description_share}/urdf/slambot.ros2_control.xacro"/>
   <xacro:include filename="${slambot_description_share}/urdf/slambot_urdf.gazebo"/>
 <link name="base_footprint"/>
@@ -14,4 +13,5 @@
   <inertial>
     <origin xyz="0.005119635718873044 -0.00011101592777540043 0.08162335600373799" rpy="0 0 0"/>
+    <!-- <mass value="3.0305928330495275"/> -->
     <mass value="3.0305928330495275"/>
     <inertia ixx="0.013459" iyy="0.014737" izz="0.007942" ixy="5e-06" iyz="-2.9e-05" ixz="0.000775"/>
