Commit message: Update

File: src/slambot_description/urdf/slambot.ros2_control.xacro (robot description, xacro)
@@ -1,4 +1,4 @@
 <?xml version="1.0" ?>
-<robot name="slambot_urdf" xmlns:xacro="http://www.ros.org/wiki/xacro">
+<robot xmlns:xacro="http://www.ros.org/wiki/xacro">
     <ros2_control name="Slambot" type="system">
         <!-- <hardware>

File: src/slambot_description/urdf/slambot_gz_urdf.xacro (robot description, xacro)
@@ -4,5 +4,8 @@
                   value="$(find slambot_description)"/>
   <xacro:include filename="${slambot_description_share}/urdf/materials.xacro"/>
+  <xacro:include filename="${slambot_description_share}/urdf/common_properties.xacro"/>
   <xacro:include filename="${slambot_description_share}/urdf/slambot_urdf.gazebo"/>
+  <xacro:include filename="${slambot_description_share}/urdf/sensors.xacro"/>
+  <xacro:include filename="${slambot_description_share}/urdf/gz_plugins.xacro"/>
 <link name="base_footprint"/>
 <joint name="base_footprint_joint" type="fixed">
@@ -13,5 +16,4 @@
   <inertial>
     <origin xyz="0.005119635718873044 -0.00011101592777540043 0.08162335600373799" rpy="0 0 0"/>
-    <!-- <mass value="3.0305928330495275"/> -->
     <mass value="3.0305928330495275"/>
     <inertia ixx="0.013459" iyy="0.014737" izz="0.007942" ixy="5e-06" iyz="-2.9e-05" ixz="0.000775"/>
@@ -20,5 +22,5 @@
     <origin xyz="0 0 0" rpy="0 0 0"/>
     <geometry>
-      <mesh filename="package://slambot_description/meshes/base_link.stl" scale="0.001 0.001 0.001"/>
+      <mesh filename="${slambot_description_share}/meshes/base_link.stl" scale="0.001 0.001 0.001"/>
     </geometry>
     <material name="silver"/>
@@ -27,5 +29,5 @@
     <origin xyz="0 0 0" rpy="0 0 0"/>
     <geometry>
-      <mesh filename="package://slambot_description/meshes/base_link.stl" scale="0.001 0.001 0.001"/>
+      <mesh filename="${slambot_description_share}/meshes/base_link.stl" scale="0.001 0.001 0.001"/>
     </geometry>
   </collision>
@@ -40,5 +42,5 @@
     <origin xyz="-0.000388 -0.035625 -0.018348" rpy="0 0 0"/>
     <geometry>
-      <mesh filename="package://slambot_description/meshes/Wheel2_1.stl" scale="0.001 0.001 0.001"/>
+      <mesh filename="${slambot_description_share}/meshes/Wheel2_1.stl" scale="0.001 0.001 0.001"/>
     </geometry>
     <material name="silver"/>
@@ -47,5 +49,5 @@
     <origin xyz="-0.000388 -0.035625 -0.018348" rpy="0 0 0"/>
     <geometry>
-      <mesh filename="package://slambot_description/meshes/Wheel2_1.stl" scale="0.001 0.001 0.001"/>
+      <mesh filename="${slambot_description_share}/meshes/Wheel2_1.stl" scale="0.001 0.001 0.001"/>
     </geometry>
   </collision>
@@ -60,5 +62,5 @@
     <origin xyz="-0.000387 0.036475 -0.018348" rpy="0 0 0"/>
     <geometry>
-      <mesh filename="package://slambot_description/meshes/Wheel1_1.stl" scale="0.001 0.001 0.001"/>
+      <mesh filename="${slambot_description_share}/meshes/Wheel1_1.stl" scale="0.001 0.001 0.001"/>
     </geometry>
     <material name="silver"/>
@@ -67,5 +69,5 @@
     <origin xyz="-0.000387 0.036475 -0.018348" rpy="0 0 0"/>
     <geometry>
-      <mesh filename="package://slambot_description/meshes/Wheel1_1.stl" scale="0.001 0.001 0.001"/>
+      <mesh filename="${slambot_description_share}/meshes/Wheel1_1.stl" scale="0.001 0.001 0.001"/>
     </geometry>
   </collision>

File: src/slambot_description/urdf/slambot_urdf.xacro (robot description, xacro)
@@ -6,4 +6,5 @@
   <xacro:include filename="${slambot_description_share}/urdf/slambot.ros2_control.xacro"/>
   <xacro:include filename="${slambot_description_share}/urdf/slambot_urdf.gazebo"/>
+  <!-- <xacro:include filename="${slambot_description_share}/urdf/sensors.xacro"/> -->
 <link name="base_footprint"/>
 <joint name="base_footprint_joint" type="fixed">
