Commit message: Changes to return to the mini robot

File: src/tank_description/urdf/gz_plugins.xacro (robot description, xacro)
@@ -17,5 +17,5 @@
    </plugin>
 </gazebo>
-<gazebo reference="camera_link">
+<!-- <gazebo reference="camera_link">
    <sensor name="camera" type="camera">
       <camera>
@@ -42,4 +42,33 @@
       <visualize>true</visualize>
       <topic>camera/image_raw</topic>
+   </sensor>
+</gazebo> -->
+<gazebo reference="camera_link">
+   <sensor name="camera" type="depth">
+      <camera>
+         <horizontal_fov>1.3962634</horizontal_fov>
+         <image>
+            <width>640</width>
+            <height>480</height>
+            <format>B8G8R8</format>
+         </image>
+         <clip>
+            <near>0.1</near>
+            <far>15</far>
+         </clip>
+         <noise>
+            <type>gaussian</type>
+            <mean>0.0</mean>
+            <stddev>0.007</stddev>
+         </noise>
+         <optical_frame_id>camera_optical_link</optical_frame_id>
+         <camera_info_topic>camera/camera_info</camera_info_topic>
+      </camera>
+      <always_on>1</always_on>
+      <update_rate>30</update_rate>
+      <visualize>true</visualize>
+      <topic>camera/image_raw</topic>
+      <min_depth></min_depth>
+      <max_depth></max_depth>
    </sensor>
 </gazebo>

File: src/tank_description/urdf/tank.ros2_control.xacro (robot description, xacro)
@@ -10,5 +10,5 @@
            <param name="left_wheel_name">left_back_wheel_joint</param>
            <param name="right_wheel_name">right_back_wheel_joint</param>
-           <param name="loop_rate">200</param>
+           <param name="loop_rate">100</param>
            <param name="device">/dev/ttyUSB0</param>
            <param name="baud_rate">115200</param>
@@ -18,11 +18,11 @@
         <joint name="left_back_wheel_joint">
             <command_interface name="velocity"/>
+            <state_interface name="position"/>
             <state_interface name="velocity"/>
+        </joint>
+        <joint name="right_back_wheel_joint">
+            <command_interface name="velocity"/>
             <state_interface name="position"/>
-        </joint>
-            <joint name="right_back_wheel_joint">
-            <command_interface name="velocity"/>
             <state_interface name="velocity"/>
-            <state_interface name="position"/>
         </joint>
     </ros2_control>

File: src/tank_description/urdf/tank_urdf.xacro (robot description, xacro)
@@ -4,5 +4,5 @@
                   value="$(find tank_description)"/>
   <xacro:include filename="${tank_description_share}/urdf/tank.ros2_control.xacro"/>
-  <xacro:include filename="${tank_description_share}/urdf/tank.common_properties.xacro"/>
+  <xacro:include filename="${tank_description_share}/urdf/common_properties.xacro"/>
   <xacro:include filename="${tank_description_share}/urdf/sensors.xacro"/>
   <xacro:property name="wheel_mass" value="5"/>
